File: kicad6/GH60_Template.kicad_pcb (KiCad board)
At the start: 2 copper layers, 285 x 94.6 mm, 69 parts, among them J3 hole1plate, J4 hole2plate, J5 hole2plate, J6 hole2plate, J7 hole3plate, J8 hole3plate, SW1 SW_PUSH, SW10 SW_PUSH, SW11 SW_PUSH, SW12 SW_PUSH, SW13 SW_PUSH, SW14 SW_PUSH, SW15 SW_PUSH, SW16 SW_PUSH, SW17 SW_PUSH, SW18 SW_PUSH, SW19 SW_PUSH, SW2 KEY_SWITCH, SW20 SW_PUSH, SW21 SW_PUSH, SW22 SW_PUSH, SW23 SW_PUSH, SW24 SW_PUSH, SW25 SW_PUSH, SW26 SW_PUSH, SW27 SW_PUSH, SW28 SW_PUSH, SW29 SW_PUSH, SW3 SW_PUSH, SW30 SW_PUSH, SW31 SW_PUSH, SW32 SW_PUSH, SW33 SW_PUSH, SW34 SW_PUSH, SW35 SW_PUSH, SW36 SW_PUSH, SW37 SW_PUSH, SW38 SW_PUSH, SW39 SW_PUSH, SW4 KEY_SWITCH, SW40 SW_PUSH, SW41 SW_PUSH, SW42 SW_PUSH, SW43 SW_PUSH, SW44 SW_PUSH, SW45 SW_PUSH, SW46 SW_PUSH, SW47 SW_PUSH, SW48 SW_PUSH, SW49 SW_PUSH, SW5 SW_PUSH, SW50 SW_PUSH, SW51 SW_PUSH, SW52 SW_PUSH, SW53 SW_PUSH, SW54 SW_PUSH, SW55 SW_PUSH, SW56 SW_PUSH, SW57 SW_PUSH, SW58 SW_PUSH, SW59 SW_PUSH, SW6 SW_PUSH, SW60 SW_PUSH, SW61 SW_PUSH, SW7 SW_PUSH, SW8 SW_PUSH, SW9 SW_PUSH, U2 5077CR-16-SMC2-BK-TR

Commit message: Add the footprint
Parts:
- moved J5 0.12 mm to (152.0, 71.5)
- moved J6 0.12 mm to (214.3, 109.7)
- moved J7 0.12 mm to (25.3, 81.0)
- moved J8 0.12 mm to (307.3, 81.0)
- moved J3 0.12 mm to (49.0, 52.4)
- moved J4 0.12 mm to (283.8, 52.4)
- moved U2 0.12 mm to (42.0, 29.6)
- moved SWR1 0.12 mm to (49.7, 70.5)
Changed lines of the file:
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@@
   )
   (footprint "footprints:hole2plate" (layer "F.Cu")
-    (at 214.2994 109.59445)
+    (at 214.2994 109.71445)
     (attr exclude_from_pos_files exclude_from_bom)
     (fp_text reference "J6" (at 0 -2.16 unlocked) (layer "F.SilkS") hide
@@
   )
   (footprint "footprints:hole2plate" (layer "F.Cu")
-    (at 152 71.39375)
+    (at 152 71.51375)
     (attr exclude_from_pos_files exclude_from_bom)
     (fp_text reference "J5" (at 0 -2.16 unlocked) (layer "F.SilkS") hide
@@
   )
   (footprint "footprints:hole2plate" (layer "F.Cu")
-    (at 283.8499 52.29455)
+    (at 283.8499 52.41455)
     (attr exclude_from_pos_files exclude_from_bom)
     (fp_text reference "J4" (at 0 -2.16 unlocked) (layer "F.SilkS") hide
@@
   )
   (footprint "footprints:hole1plate" (layer "F.Cu")
-    (at 48.9993 52.29455)
+    (at 48.9993 52.41455)
     (attr exclude_from_pos_files exclude_from_bom)
     (fp_text reference "J3" (at 0 -2.06 unlocked) (layer "F.SilkS") hide
@@
   )
   (footprint "footprints:hole3plate" (layer "F.Cu")
-    (at 307.3412 80.89495)
+    (at 307.3412 81.01495)
     (attr exclude_from_pos_files exclude_from_bom)
     (fp_text reference "J8" (at 0 -2.16 unlocked) (layer "F.SilkS") hide
@@
   )
   (footprint "footprints:hole3plate" (layer "F.Cu")
-    (at 25.2589 80.89495)
+    (at 25.2589 81.01495)
     (attr exclude_from_pos_files exclude_from_bom)
     (fp_text reference "J7" (at 0 -2.16 unlocked) (layer "F.SilkS") hide
@@
   )
   (footprint "footprints:connector_usb2c_5077CR-16-SMC2-BK-TR" (layer "B.Cu")
-    (at 42 29.5238)
+    (at 42 29.6438)
     (fp_text reference "U2" (at 0 1.67 180 unlocked) (layer "B.SilkS") hide
       (effects (font (size 0.5 0.5) (thickness 0.075)) (justify mirror))
@@
   )
   (footprint "Button_Switch_THT:SW_PUSH_6mm" (layer "B.Cu")
-    (at 49.701 70.34175 -90)
+    (at 49.701 70.46175 -90)
     (descr "https://www.omron.com/ecb/products/pdf/en-b3f.pdf")
     (tags "tact sw push 6mm")
@@
     )
   )
-  (gr_arc (start 306.8 24.39375) (mid 308.214246 24.979519) (end 308.8 26.39375) (layer "Edge.Cuts") (width 0.1))
-  (gr_arc (start 23.8 26.39375) (mid 24.385789 24.979554) (end 25.8 24.39375) (layer "Edge.Cuts") (width 0.1))
-  (gr_arc (start 25.8 118.99615) (mid 24.385754 118.410381) (end 23.8 116.99615) (layer "Edge.Cuts") (width 0.1))
-  (gr_line (start 25.8 118.99615) (end 306.8 118.99615) (layer "Edge.Cuts") (width 0.1))
-  (gr_line (start 306.8 24.39375) (end 25.8 24.39375) (layer "Edge.Cuts") (width 0.1))
-  (gr_arc (start 308.8 116.99615) (mid 308.214211 118.410346) (end 306.8 118.99615) (layer "Edge.Cuts") (width 0.1))
-  (gr_line (start 308.8 116.99615) (end 308.8 26.39375) (layer "Edge.Cuts") (width 0.1))
-  (gr_line (start 23.8 26.39375) (end 23.8 116.99615) (layer "Edge.Cuts") (width 0.1))
+  (gr_arc (start 306.8 24.51375) (mid 308.214261 25.099504) (end 308.8 26.51375) (layer "Edge.Cuts") (width 0.1))
+  (gr_arc (start 23.8 26.51375) (mid 24.385804 25.099569) (end 25.8 24.51375) (layer "Edge.Cuts") (width 0.1))
+  (gr_arc (start 25.8 119.11615) (mid 24.385739 118.530396) (end 23.8 117.11615) (layer "Edge.Cuts") (width 0.1))
+  (gr_line (start 25.8 119.11615) (end 306.8 119.11615) (layer "Edge.Cuts") (width 0.1))
+  (gr_line (start 306.8 24.51375) (end 25.8 24.51375) (layer "Edge.Cuts") (width 0.1))
+  (gr_arc (start 308.8 117.11615) (mid 308.214196 118.530331) (end 306.8 119.11615) (layer "Edge.Cuts") (width 0.1))
+  (gr_line (start 308.8 117.11615) (end 308.8 26.51375) (layer "Edge.Cuts") (width 0.1))
+  (gr_line (start 23.8 26.51375) (end 23.8 117.11615) (layer "Edge.Cuts") (width 0.1))
   (gr_text "Please remove U2 (USB Connector) and SWR1 (Reset Switch) if you're making the switch plate.\nDon't move screw holes!" (at 23.8125 16.66875) (layer "Cmts.User")
     (effects (font (size 2 2) (thickness 0.4)) (justify left))

Commit message: Added footprints
Parts:
- J3: value hole1plate -> hole_poker1_edge; footprint footprints:hole1plate -> footprints:hole_poker1_edge
- J4, J5, J6: value hole2plate -> hole_poker2_edge; footprint footprints:hole2plate -> footprints:hole_poker2_edge
- J7, J8: value hole3plate -> hole_poker3_edge; footprint footprints:hole3plate -> footprints:hole_poker3_edge
Changed lines of the file:
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@@
     (fp_line (start -11.90625 -9.525) (end -11.90625 9.525) (layer "F.Fab") (width 0.15))
   )
-  (footprint "footprints:hole2plate" (layer "F.Cu")
+  (footprint "footprints:hole_poker2_edge" (layer "F.Cu")
     (at 214.2994 109.71445)
-    (attr exclude_from_pos_files exclude_from_bom)
+    (attr board_only exclude_from_pos_files exclude_from_bom)
     (fp_text reference "J6" (at 0 -2.16 unlocked) (layer "F.SilkS") hide
       (effects (font (size 1 1) (thickness 0.15)))
     )
-    (fp_text value "hole2plate" (at 0 2.244 unlocked) (layer "F.SilkS") hide
-      (effects (font (size 1 1) (thickness 0.15)))
-    )
-    (fp_line (start -1.25095 -1.24968) (end 1.25095 -1.24968) (layer "Edge.Cuts") (width 0.15))
-    (fp_line (start -1.25095 1.24968) (end 1.25095 1.24968) (layer "Edge.Cuts") (width 0.15))
-    (fp_arc (start 1.25095 -1.24968) (mid 2.50063 0) (end 1.25095 1.24968) (layer "Edge.Cuts") (width 0.15))
-    (fp_arc (start -1.25095 1.24968) (mid -2.50063 0) (end -1.25095 -1.24968) (layer "Edge.Cuts") (width 0.15))
-  )
-  (footprint "footprints:hole2plate" (layer "F.Cu")
-    (at 152 71.51375)
-    (attr exclude_from_pos_files exclude_from_bom)
-    (fp_text reference "J5" (at 0 -2.16 unlocked) (layer "F.SilkS") hide
-      (effects (font (size 1 1) (thickness 0.15)))
-    )
-    (fp_text value "hole2plate" (at 0 2.244 unlocked) (layer "F.SilkS") hide
+    (fp_text value "hole_poker2_edge" (at 0 2.244 unlocked) (layer "F.SilkS") hide
       (effects (font (size 1 1) (thickness 0.15)))
     )
@@
     (fp_arc (start 1.25095 -1.24968) (mid 2.50063 0) (end 1.25095 1.24968) (layer "Edge.Cuts") (width 0.15))
   )
-  (footprint "footprints:hole2plate" (layer "F.Cu")
+  (footprint "footprints:hole_poker2_edge" (layer "F.Cu")
+    (at 152 71.51375)
+    (attr board_only exclude_from_pos_files exclude_from_bom)
+    (fp_text reference "J5" (at 0 -2.16 unlocked) (layer "F.SilkS") hide
+      (effects (font (size 1 1) (thickness 0.15)))
+    )
+    (fp_text value "hole_poker2_edge" (at 0 2.244 unlocked) (layer "F.SilkS") hide
+      (effects (font (size 1 1) (thickness 0.15)))
+    )
+    (fp_line (start -1.25095 1.24968) (end 1.25095 1.24968) (layer "Edge.Cuts") (width 0.15))
+    (fp_line (start -1.25095 -1.24968) (end 1.25095 -1.24968) (layer "Edge.Cuts") (width 0.15))
+    (fp_arc (start -1.25095 1.24968) (mid -2.50063 0) (end -1.25095 -1.24968) (layer "Edge.Cuts") (width 0.15))
+    (fp_arc (start 1.25095 -1.24968) (mid 2.50063 0) (end 1.25095 1.24968) (layer "Edge.Cuts") (width 0.15))
+  )
+  (footprint "footprints:hole_poker2_edge" (layer "F.Cu")
     (at 283.8499 52.41455)
-    (attr exclude_from_pos_files exclude_from_bom)
+    (attr board_only exclude_from_pos_files exclude_from_bom)
     (fp_text reference "J4" (at 0 -2.16 unlocked) (layer "F.SilkS") hide
       (effects (font (size 1 1) (thickness 0.15)))
     )
-    (fp_text value "hole2plate" (at 0 2.244 unlocked) (layer "F.SilkS") hide
+    (fp_text value "hole_poker2_edge" (at 0 2.244 unlocked) (layer "F.SilkS") hide
       (effects (font (size 1 1) (thickness 0.15)))
     )
+    (fp_line (start -1.25095 1.24968) (end 1.25095 1.24968) (layer "Edge.Cuts") (width 0.15))
     (fp_line (start -1.25095 -1.24968) (end 1.25095 -1.24968) (layer "Edge.Cuts") (width 0.15))
-    (fp_line (start -1.25095 1.24968) (end 1.25095 1.24968) (layer "Edge.Cuts") (width 0.15))
+    (fp_arc (start 1.25095 -1.24968) (mid 2.50063 0) (end 1.25095 1.24968) (layer "Edge.Cuts") (width 0.15))
     (fp_arc (start -1.25095 1.24968) (mid -2.50063 0) (end -1.25095 -1.24968) (layer "Edge.Cuts") (width 0.15))
-    (fp_arc (start 1.25095 -1.24968) (mid 2.50063 0) (end 1.25095 1.24968) (layer "Edge.Cuts") (width 0.15))
   )
-  (footprint "footprints:hole1plate" (layer "F.Cu")
+  (footprint "footprints:hole_poker1_edge" (layer "F.Cu")
     (at 48.9993 52.41455)
-    (attr exclude_from_pos_files exclude_from_bom)
+    (attr board_only exclude_from_pos_files exclude_from_bom)
     (fp_text reference "J3" (at 0 -2.06 unlocked) (layer "F.SilkS") hide
       (effects (font (size 1 1) (thickness 0.15)))
     )
-    (fp_text value "hole1plate" (at 0 2.144 unlocked) (layer "F.SilkS") hide
+    (fp_text value "hole_poker1_edge" (at 0 2.144 unlocked) (layer "F.SilkS") hide
       (effects (font (size 1 1) (thickness 0.15)))
     )
     (fp_circle (center 0 0) (end 1.2497 0) (layer "Edge.Cuts") (width 0.15) (fill none))
   )
-  (footprint "footprints:hole3plate" (layer "F.Cu")
+  (footprint "footprints:hole_poker3_edge" (layer "F.Cu")
     (at 307.3412 81.01495)
-    (attr exclude_from_pos_files exclude_from_bom)
+    (attr board_only exclude_from_pos_files exclude_from_bom)
     (fp_text reference "J8" (at 0 -2.16 unlocked) (layer "F.SilkS") hide
       (effects (font (size 1 1) (thickness 0.15)))
     )
-    (fp_text value "hole3plate" (at 0 2.244 unlocked) (layer "F.SilkS") hide
+    (fp_text value "hole_poker3_edge" (at 0 2.244 unlocked) (layer "F.SilkS") hide
       (effects (font (size 1 1) (thickness 0.15)))
     )
+    (fp_line (start -2.25044 1.24968) (end 2.25044 1.24968) (layer "Edge.Cuts") (width 0.15))
     (fp_line (start -2.25044 -1.24968) (end 2.25044 -1.24968) (layer "Edge.Cuts") (width 0.15))
-    (fp_line (start -2.25044 1.24968) (end 2.25044 1.24968) (layer "Edge.Cuts") (width 0.15))
+    (fp_arc (start 2.25044 -1.24968) (mid 3.50012 0) (end 2.25044 1.24968) (layer "Edge.Cuts") (width 0.15))
     (fp_arc (start -2.25044 1.24968) (mid -3.50012 0) (end -2.25044 -1.24968) (layer "Edge.Cuts") (width 0.15))
-    (fp_arc (start 2.25044 -1.24968) (mid 3.50012 0) (end 2.25044 1.24968) (layer "Edge.Cuts") (width 0.15))
   )
-  (footprint "footprints:hole3plate" (layer "F.Cu")
+  (footprint "footprints:hole_poker3_edge" (layer "F.Cu")
     (at 25.2589 81.01495)
-    (attr exclude_from_pos_files exclude_from_bom)
+    (attr board_only exclude_from_pos_files exclude_from_bom)
     (fp_text reference "J7" (at 0 -2.16 unlocked) (layer "F.SilkS") hide
       (effects (font (size 1 1) (thickness 0.15)))
     )
-    (fp_text value "hole3plate" (at 0 2.244 unlocked) (layer "F.SilkS") hide
+    (fp_text value "hole_poker3_edge" (at 0 2.244 unlocked) (layer "F.SilkS") hide
       (effects (font (size 1 1) (thickness 0.15)))
     )

Commit message: 1. (PCB) All items except MX switches offset Y axis -0.4 mm. 2. All footprints have moved to Jun_footprints (other repository).
Parts:
- J3: footprint footprints:hole_poker1_edge -> Jun_footprints:hole_poker1_edge
- J4, J5, J6: footprint footprints:hole_poker2_edge -> Jun_footprints:hole_poker2_edge
- J7, J8: footprint footprints:hole_poker3_edge -> Jun_footprints:hole_poker3_edge
- U2: footprint footprints:connector_usb2c_5077CR-16-SMC2-BK-TR -> Jun_footprints:connector_usb2c_5077CR-16-SMC2-BK-TR
- moved J5 0.40 mm to (152.0, 71.1)
- moved J6 0.40 mm to (214.3, 109.3)
- moved J7 0.40 mm to (25.3, 80.6)
- moved J8 0.40 mm to (307.3, 80.6)
- moved J3 0.40 mm to (49.0, 52.0)
- moved J4 0.40 mm to (283.8, 52.0)
- moved U2 0.40 mm to (42.0, 29.2)
- moved SWR1 0.40 mm to (49.7, 70.1)
Changed lines of the file:
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@@
     (fp_line (start -11.90625 -9.525) (end -11.90625 9.525) (layer "F.Fab") (width 0.15))
   )
-  (footprint "footprints:hole_poker2_edge" (layer "F.Cu")
-    (at 214.2994 109.71445)
+  (footprint "Jun_footprints:hole_poker2_edge" (layer "F.Cu")
+    (at 214.2994 109.31445)
     (attr board_only exclude_from_pos_files exclude_from_bom)
     (fp_text reference "J6" (at 0 -2.16 unlocked) (layer "F.SilkS") hide
@@
     (fp_arc (start 1.25095 -1.24968) (mid 2.50063 0) (end 1.25095 1.24968) (layer "Edge.Cuts") (width 0.15))
   )
-  (footprint "footprints:hole_poker2_edge" (layer "F.Cu")
-    (at 152 71.51375)
+  (footprint "Jun_footprints:hole_poker2_edge" (layer "F.Cu")
+    (at 152 71.11375)
     (attr board_only exclude_from_pos_files exclude_from_bom)
     (fp_text reference "J5" (at 0 -2.16 unlocked) (layer "F.SilkS") hide
@@
     (fp_arc (start 1.25095 -1.24968) (mid 2.50063 0) (end 1.25095 1.24968) (layer "Edge.Cuts") (width 0.15))
   )
-  (footprint "footprints:hole_poker2_edge" (layer "F.Cu")
-    (at 283.8499 52.41455)
+  (footprint "Jun_footprints:hole_poker2_edge" (layer "F.Cu")
+    (at 283.8499 52.01455)
     (attr board_only exclude_from_pos_files exclude_from_bom)
     (fp_text reference "J4" (at 0 -2.16 unlocked) (layer "F.SilkS") hide
@@
     (fp_arc (start -1.25095 1.24968) (mid -2.50063 0) (end -1.25095 -1.24968) (layer "Edge.Cuts") (width 0.15))
   )
-  (footprint "footprints:hole_poker1_edge" (layer "F.Cu")
-    (at 48.9993 52.41455)
+  (footprint "Jun_footprints:hole_poker1_edge" (layer "F.Cu")
+    (at 48.9993 52.01455)
     (attr board_only exclude_from_pos_files exclude_from_bom)
     (fp_text reference "J3" (at 0 -2.06 unlocked) (layer "F.SilkS") hide
@@
     (fp_circle (center 0 0) (end 1.2497 0) (layer "Edge.Cuts") (width 0.15) (fill none))
   )
-  (footprint "footprints:hole_poker3_edge" (layer "F.Cu")
-    (at 307.3412 81.01495)
+  (footprint "Jun_footprints:hole_poker3_edge" (layer "F.Cu")
+    (at 307.3412 80.61495)
     (attr board_only exclude_from_pos_files exclude_from_bom)
     (fp_text reference "J8" (at 0 -2.16 unlocked) (layer "F.SilkS") hide
@@
     (fp_arc (start -2.25044 1.24968) (mid -3.50012 0) (end -2.25044 -1.24968) (layer "Edge.Cuts") (width 0.15))
   )
-  (footprint "footprints:hole_poker3_edge" (layer "F.Cu")
-    (at 25.2589 81.01495)
+  (footprint "Jun_footprints:hole_poker3_edge" (layer "F.Cu")
+    (at 25.2589 80.61495)
     (attr board_only exclude_from_pos_files exclude_from_bom)
     (fp_text reference "J7" (at 0 -2.16 unlocked) (layer "F.SilkS") hide
@@
     (fp_arc (start 2.25044 -1.24968) (mid 3.50012 0) (end 2.25044 1.24968) (layer "Edge.Cuts") (width 0.15))
   )
-  (footprint "footprints:connector_usb2c_5077CR-16-SMC2-BK-TR" (layer "B.Cu")
-    (at 42 29.6438)
+  (footprint "Jun_footprints:connector_usb2c_5077CR-16-SMC2-BK-TR" (layer "B.Cu")
+    (at 42 29.2438)
     (fp_text reference "U2" (at 0 1.67 180 unlocked) (layer "B.SilkS") hide
       (effects (font (size 0.5 0.5) (thickness 0.075)) (justify mirror))
@@
   )
   (footprint "Button_Switch_THT:SW_PUSH_6mm" (layer "B.Cu")
-    (at 49.701 70.46175 -90)
+    (at 49.701 70.06175 -90)
     (descr "https://www.omron.com/ecb/products/pdf/en-b3f.pdf")
     (tags "tact sw push 6mm")
@@
     )
   )
-  (gr_arc (start 306.8 24.51375) (mid 308.214261 25.099504) (end 308.8 26.51375) (layer "Edge.Cuts") (width 0.1))
-  (gr_arc (start 23.8 26.51375) (mid 24.385804 25.099569) (end 25.8 24.51375) (layer "Edge.Cuts") (width 0.1))
-  (gr_arc (start 25.8 119.11615) (mid 24.385739 118.530396) (end 23.8 117.11615) (layer "Edge.Cuts") (width 0.1))
-  (gr_line (start 25.8 119.11615) (end 306.8 119.11615) (layer "Edge.Cuts") (width 0.1))
-  (gr_line (start 306.8 24.51375) (end 25.8 24.51375) (layer "Edge.Cuts") (width 0.1))
-  (gr_arc (start 308.8 117.11615) (mid 308.214196 118.530331) (end 306.8 119.11615) (layer "Edge.Cuts") (width 0.1))
-  (gr_line (start 308.8 117.11615) (end 308.8 26.51375) (layer "Edge.Cuts") (width 0.1))
-  (gr_line (start 23.8 26.51375) (end 23.8 117.11615) (layer "Edge.Cuts") (width 0.1))
+  (gr_arc (start 306.8 24.11375) (mid 308.214225 24.69951) (end 308.8 26.11375) (layer "Edge.Cuts") (width 0.1))
+  (gr_arc (start 23.8 26.11375) (mid 24.385813 24.699563) (end 25.8 24.11375) (layer "Edge.Cuts") (width 0.1))
+  (gr_arc (start 25.8 118.71615) (mid 24.385775 118.13039) (end 23.8 116.71615) (layer "Edge.Cuts") (width 0.1))
+  (gr_line (start 25.8 118.71615) (end 306.8 118.71615) (layer "Edge.Cuts") (width 0.1))
+  (gr_line (start 306.8 24.11375) (end 25.8 24.11375) (layer "Edge.Cuts") (width 0.1))
+  (gr_arc (start 308.8 116.71615) (mid 308.214202 118.130367) (end 306.8 118.71615) (layer "Edge.Cuts") (width 0.1))
+  (gr_line (start 308.8 116.71615) (end 308.8 26.11375) (layer "Edge.Cuts") (width 0.1))
+  (gr_line (start 23.8 26.11375) (end 23.8 116.71615) (layer "Edge.Cuts") (width 0.1))
   (gr_text "Please remove U2 (USB Connector) and SWR1 (Reset Switch) if you're making the switch plate.\nDon't move screw holes!" (at 23.8125 16.66875) (layer "Cmts.User")
     (effects (font (size 2 2) (thickness 0.4)) (justify left))
