File: kicad6/GH60_Template.kicad_sch (KiCad schematic)
At the start: 253 parts, among them J1 Conn_01x02, J2 Conn_01x04, J3 Conn_01x01, J4 Conn_01x01, J5 Conn_01x01, J6 Conn_01x01, J7 Conn_01x01, J8 Conn_01x01, SW1 SW_PUSH, SW10 SW_PUSH, SW11 SW_PUSH, SW12 SW_PUSH, SW13 SW_PUSH, SW14 SW_PUSH, SW15 SW_PUSH, SW16 SW_PUSH, SW17 SW_PUSH, SW18 SW_PUSH, SW19 SW_PUSH, SW2 SW_PUSH, SW20 SW_PUSH, SW21 SW_PUSH, SW22 SW_PUSH, SW23 SW_PUSH, SW24 SW_PUSH, SW25 SW_PUSH, SW26 SW_PUSH, SW27 SW_PUSH, SW28 SW_PUSH, SW29 SW_PUSH, SW3 SW_PUSH, SW30 SW_PUSH, SW31 SW_PUSH, SW32 SW_PUSH, SW33 SW_PUSH, SW34 SW_PUSH, SW35 SW_PUSH, SW36 SW_PUSH, SW37 SW_PUSH, SW38 SW_PUSH, SW39 SW_PUSH, SW4 SW_PUSH, SW40 SW_PUSH, SW41 SW_PUSH, SW42 SW_PUSH, SW43 SW_PUSH, SW44 SW_PUSH, SW45 SW_PUSH, SW46 SW_PUSH, SW47 SW_PUSH, SW48 SW_PUSH, SW49 SW_PUSH, SW5 SW_PUSH, SW50 SW_PUSH, SW51 SW_PUSH, SW52 SW_PUSH, SW53 SW_PUSH, SW54 SW_PUSH, SW55 SW_PUSH, SW56 SW_PUSH, SW57 SW_PUSH, SW58 SW_PUSH, SW59 SW_PUSH, SW6 SW_PUSH, SW60 SW_PUSH, SW61 SW_PUSH, SW62 SW_PUSH, SW63 SW_PUSH, SW64 SW_PUSH, SW65 SW_PUSH, SW66 SW_PUSH, SW67 SW_PUSH, SW68 SW_PUSH, SW69 SW_PUSH, SW7 SW_PUSH, SW70 SW_PUSH, SW71 SW_PUSH, SW72 SW_PUSH, SW73 SW_PUSH, SW74 SW_PUSH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

Commit message: Added footprints
Parts:
- J3: footprint footprints:hole1 -> footprints:hole_poker1_npth
- J4, J5, J6: footprint footprints:hole2 -> footprints:hole_poker2_npth
- J7, J8: footprint footprints:hole3 -> footprints:hole_poker3_npth
Changed lines of the file:
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@@
       (effects (font (size 1.27 1.27)) (justify left))
     )
-    (property "Footprint" "footprints:hole3" (id 2) (at 397.51 177.165 0)
+    (property "Footprint" "footprints:hole_poker3_npth" (id 2) (at 397.51 177.165 0)
       (effects (font (size 1.27 1.27)) hide)
     )
@@
       (effects (font (size 1.27 1.27)) (justify left))
     )
-    (property "Footprint" "footprints:hole3" (id 2) (at 397.51 182.245 0)
+    (property "Footprint" "footprints:hole_poker3_npth" (id 2) (at 397.51 182.245 0)
       (effects (font (size 1.27 1.27)) hide)
     )
@@
       (effects (font (size 1.27 1.27)) (justify left))
     )
-    (property "Footprint" "footprints:hole2" (id 2) (at 397.51 167.005 0)
+    (property "Footprint" "footprints:hole_poker2_npth" (id 2) (at 397.51 167.005 0)
       (effects (font (size 1.27 1.27)) hide)
     )
@@
       (effects (font (size 1.27 1.27)) (justify left))
     )
-    (property "Footprint" "footprints:hole2" (id 2) (at 397.51 172.085 0)
+    (property "Footprint" "footprints:hole_poker2_npth" (id 2) (at 397.51 172.085 0)
       (effects (font (size 1.27 1.27)) hide)
     )
@@
       (effects (font (size 1.27 1.27)) (justify left))
     )
-    (property "Footprint" "footprints:hole1" (id 2) (at 397.51 156.845 0)
+    (property "Footprint" "footprints:hole_poker1_npth" (id 2) (at 397.51 156.845 0)
       (effects (font (size 1.27 1.27)) hide)
     )
@@
       (effects (font (size 1.27 1.27)) (justify left))
     )
-    (property "Footprint" "footprints:hole2" (id 2) (at 397.51 161.925 0)
+    (property "Footprint" "footprints:hole_poker2_npth" (id 2) (at 397.51 161.925 0)
       (effects (font (size 1.27 1.27)) hide)
     )
@@
     )
     (path "/00000000-0000-0000-0000-000064540388"
-      (reference "J3") (unit 1) (value "Conn_01x01") (footprint "footprints:hole1")
+      (reference "J3") (unit 1) (value "Conn_01x01") (footprint "footprints:hole_poker1_npth")
     )
     (path "/00000000-0000-0000-0000-00006454039c"
-      (reference "J4") (unit 1) (value "Conn_01x01") (footprint "footprints:hole2")
+      (reference "J4") (unit 1) (value "Conn_01x01") (footprint "footprints:hole_poker2_npth")
     )
     (path "/00000000-0000-0000-0000-0000629102f3"
-      (reference "J5") (unit 1) (value "Conn_01x01") (footprint "footprints:hole2")
+      (reference "J5") (unit 1) (value "Conn_01x01") (footprint "footprints:hole_poker2_npth")
     )
     (path "/00000000-0000-0000-0000-00006291030e"
-      (reference "J6") (unit 1) (value "Conn_01x01") (footprint "footprints:hole2")
+      (reference "J6") (unit 1) (value "Conn_01x01") (footprint "footprints:hole_poker2_npth")
     )
     (path "/00000000-0000-0000-0000-00005cc48ceb"
-      (reference "J7") (unit 1) (value "Conn_01x01") (footprint "footprints:hole3")
+      (reference "J7") (unit 1) (value "Conn_01x01") (footprint "footprints:hole_poker3_npth")
     )
     (path "/00000000-0000-0000-0000-00005cc9ee92"
-      (reference "J8") (unit 1) (value "Conn_01x01") (footprint "footprints:hole3")
+      (reference "J8") (unit 1) (value "Conn_01x01") (footprint "footprints:hole_poker3_npth")
     )
     (path "/00000000-0000-0000-0000-00005cafbd59"

Commit message: 1. (PCB) All items except MX switches offset Y axis -0.4 mm. 2. All footprints have moved to Jun_footprints (other repository).
Parts:
- J2: footprint footprints:jumper_usb2 -> Jun_footprints:jumper_usb2_10.1x10.3
- J3: footprint footprints:hole_poker1_npth -> Jun_footprints:hole_poker1_npth
- J4, J5, J6: footprint footprints:hole_poker2_npth -> Jun_footprints:hole_poker2_npth
- J7, J8: footprint footprints:hole_poker3_npth -> Jun_footprints:hole_poker3_npth
- U2: footprint footprints:connector_usb2c_5077CR-16-SMC2-BK-TR -> Jun_footprints:connector_usb2c_5077CR-16-SMC2-BK-TR
Changed lines of the file:
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@@
       (effects (font (size 1.27 1.27)) (justify left))
     )
-    (property "Footprint" "footprints:hole_poker3_npth" (id 2) (at 397.51 177.165 0)
+    (property "Footprint" "Jun_footprints:hole_poker3_npth" (id 2) (at 397.51 177.165 0)
       (effects (font (size 1.27 1.27)) hide)
     )
@@
       (effects (font (size 1.27 1.27)) (justify left))
     )
-    (property "Footprint" "footprints:hole_poker3_npth" (id 2) (at 397.51 182.245 0)
+    (property "Footprint" "Jun_footprints:hole_poker3_npth" (id 2) (at 397.51 182.245 0)
       (effects (font (size 1.27 1.27)) hide)
     )
@@
       (effects (font (size 1.27 1.27)) (justify left))
     )
-    (property "Footprint" "footprints:hole_poker2_npth" (id 2) (at 397.51 167.005 0)
+    (property "Footprint" "Jun_footprints:hole_poker2_npth" (id 2) (at 397.51 167.005 0)
       (effects (font (size 1.27 1.27)) hide)
     )
@@
       (effects (font (size 1.27 1.27)) (justify left))
     )
-    (property "Footprint" "footprints:hole_poker2_npth" (id 2) (at 397.51 172.085 0)
+    (property "Footprint" "Jun_footprints:hole_poker2_npth" (id 2) (at 397.51 172.085 0)
       (effects (font (size 1.27 1.27)) hide)
     )
@@
       (effects (font (size 1.27 1.27)) (justify left))
     )
-    (property "Footprint" "footprints:hole_poker1_npth" (id 2) (at 397.51 156.845 0)
+    (property "Footprint" "Jun_footprints:hole_poker1_npth" (id 2) (at 397.51 156.845 0)
       (effects (font (size 1.27 1.27)) hide)
     )
@@
       (effects (font (size 1.27 1.27)) (justify left))
     )
-    (property "Footprint" "footprints:hole_poker2_npth" (id 2) (at 397.51 161.925 0)
+    (property "Footprint" "Jun_footprints:hole_poker2_npth" (id 2) (at 397.51 161.925 0)
       (effects (font (size 1.27 1.27)) hide)
     )
@@
       (effects (font (size 1.27 1.27)) (justify left))
     )
-    (property "Footprint" "footprints:jumper_usb2" (id 2) (at 378.46 115.57 0)
+    (property "Footprint" "Jun_footprints:jumper_usb2_10.1x10.3" (id 2) (at 378.46 115.57 0)
       (effects (font (size 1.27 1.27)) hide)
     )
@@
     (property "Reference" "U2" (id 0) (at 349.25 71.12 0))
     (property "Value" "USB_C_Receptacle_USB2.0" (id 1) (at 349.25 73.66 0))
-    (property "Footprint" "footprints:connector_usb2c_5077CR-16-SMC2-BK-TR" (id 2) (at 353.06 93.98 0)
+    (property "Footprint" "Jun_footprints:connector_usb2c_5077CR-16-SMC2-BK-TR" (id 2) (at 353.06 93.98 0)
       (effects (font (size 1.27 1.27)) hide)
     )
@@
     )
     (path "/5882f118-d691-4850-8b0d-6f2c3dc9ad16"
-      (reference "J2") (unit 1) (value "Conn_01x04") (footprint "footprints:jumper_usb2")
+      (reference "J2") (unit 1) (value "Conn_01x04") (footprint "Jun_footprints:jumper_usb2_10.1x10.3")
     )
     (path "/00000000-0000-0000-0000-000064540388"
-      (reference "J3") (unit 1) (value "Conn_01x01") (footprint "footprints:hole_poker1_npth")
+      (reference "J3") (unit 1) (value "Conn_01x01") (footprint "Jun_footprints:hole_poker1_npth")
     )
     (path "/00000000-0000-0000-0000-00006454039c"
-      (reference "J4") (unit 1) (value "Conn_01x01") (footprint "footprints:hole_poker2_npth")
+      (reference "J4") (unit 1) (value "Conn_01x01") (footprint "Jun_footprints:hole_poker2_npth")
     )
     (path "/00000000-0000-0000-0000-0000629102f3"
-      (reference "J5") (unit 1) (value "Conn_01x01") (footprint "footprints:hole_poker2_npth")
+      (reference "J5") (unit 1) (value "Conn_01x01") (footprint "Jun_footprints:hole_poker2_npth")
     )
     (path "/00000000-0000-0000-0000-00006291030e"
-      (reference "J6") (unit 1) (value "Conn_01x01") (footprint "footprints:hole_poker2_npth")
+      (reference "J6") (unit 1) (value "Conn_01x01") (footprint "Jun_footprints:hole_poker2_npth")
     )
     (path "/00000000-0000-0000-0000-00005cc48ceb"
-      (reference "J7") (unit 1) (value "Conn_01x01") (footprint "footprints:hole_poker3_npth")
+      (reference "J7") (unit 1) (value "Conn_01x01") (footprint "Jun_footprints:hole_poker3_npth")
     )
     (path "/00000000-0000-0000-0000-00005cc9ee92"
-      (reference "J8") (unit 1) (value "Conn_01x01") (footprint "footprints:hole_poker3_npth")
+      (reference "J8") (unit 1) (value "Conn_01x01") (footprint "Jun_footprints:hole_poker3_npth")
     )
     (path "/00000000-0000-0000-0000-00005cafbd59"
@@
     )
     (path "/af87ad17-fec6-4946-a1bf-13239f4bfde7"
-      (reference "U2") (unit 1) (value "USB_C_Receptacle_USB2.0") (footprint "footprints:connector_usb2c_5077CR-16-SMC2-BK-TR")
+      (reference "U2") (unit 1) (value "USB_C_Receptacle_USB2.0") (footprint "Jun_footprints:connector_usb2c_5077CR-16-SMC2-BK-TR")
     )
   )
